File: tests/board_samples/kicad_10/drill_types.kicad_pcb (KiCad board)
At the start: 4 copper layers, 25 x 25 mm, 3 parts

Commit message: [Tests][Workaround][KiCad 10] Restore kibot_table_drill_table group
Related to KiCad bug:
https://gitlab.com/kicad/code/kicad/-/work_items/23479

The migration removed the group used for the table
Other:
- board text added: "Reserved for table"
Changed lines of the file:
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@@
 		(layer "Edge.Cuts")
+	)
+	(gr_text "Reserved for table"
+		(at 51 58.25 0)
+		(layer "Cmts.User")
+		(effects
+			(font
+				(size 1.5 1.5)
+				(thickness 0.3)
+				(bold yes)
+			)
+			(justify left bottom)
+		)
 	)
 	(via
@@
 		(net "")
 	)
+	(group "kibot_table_drill_table"
+		(members "8f769ff7-0ab1-44a8-ac30-8af10f3c087c" "9e0d7d54-b080-48c2-a362-342413b9c768")
+	)
 	(embedded_fonts no)
