File: tests/board_samples/kicad_10/kibom-variant_3_txt.kicad_sch (KiCad schematic)
At the start: 5 parts

Commit message: [Tests][Fixed][KiCad 10] No more WRL files
Parts:
- R2: default:_3D_model ${KICAD6_3DMODEL_DIR}/Resistor_SMD.3dshapes/R_2010_5025Metric.wrl -> ${KICAD6_3DMODEL_DIR}/Resistor_SMD.3dshapes/R_2010_5025Metric.step
Changed lines of the file:
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@@
 			)
 		)
-		(property "default:_3D_model" "${KICAD6_3DMODEL_DIR}/Resistor_SMD.3dshapes/R_2010_5025Metric.wrl"
+		(property "default:_3D_model" "${KICAD6_3DMODEL_DIR}/Resistor_SMD.3dshapes/R_2010_5025Metric.step"
 			(at 63.5 43.18 0)
 			(hide yes)
