File: tests/board_samples/kicad_10/sheet_flags/sub.kicad_sch (KiCad schematic)
At the start: 1 part

Commit message: [Tests][Added] Three tests for the schematic save
- Mostly oriented to cover the sheet DNP flag
- With and without variants applied
Parts:
- R1: Config (none) -> NOR3
Changed lines of the file:
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@@
+			)
+		)
+		(property "Config" "NOR3"
+			(at 100 100 0)
+			(hide yes)
+			(show_name no)
+			(do_not_autoplace no)
+			(effects
+				(font
+					(size 1.27 1.27)
+				)
 			)
 		)
